File: PWB4000231/PWB4000231/PWB4000231.kicad_sch (KiCad schematic)
At the start: 13 parts, among them J1 Conn_02x14_Counter_Clockwise, U1 74LS375, U10 74LS74, U11 74LS74, U12 74LS157, U2 74LS157, U3 74LS244, U4 74LS04, U5 74LS375, U6 74LS157, U7 74LS74, U8 74LS21, U9 74LS157

Commit message: Moved things around to be more logically grouped
Connections:
- net PIN20: no longer U2.15 (E)
- net PIN21: no longer U9.1 (S)
- net at U5.11 (Q2): now also U6.11 (I0c), U9.6 (I1b)
- net at U5.2 (~{Q0}): now also U8.2
- net at U5.3 (Q0), U9.13 (I1d): now also U6.2 (I0a)
- net at U5.6 (~{Q1}), U8.1: no longer U9.6 (I1b)
- net +5V: now reaches U6.16 (VCC)
- net +5V: now also U2.16 (VCC)
- net UNK2: now reaches U12.2 (I0a), U2.1 (S), U8.8
- net at U4.10: now also U7.11 (C)
Other:
- moved on the sheet: J1, U1, U10A, U10B, U10C, U11A, U11B, U11C, U12, U2, U3, U4A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
